File: schematics/neurolab.kicad_pcb (KiCad board)
At the start: 2 copper layers, 164 parts, among them J1 GS3, J10 GS3, J11 GS2, J12 GS3, J13 GS3, J14 GS3, J15 GS3, J16 Channel, J17 Conn_01x02, J18 USB_OTG, J19 GS3, J2 GS3, J20 GS2, J21 GS2, J22 GS2, J23 GS2, J24 GS2, J25 GS2, J26 Conn_02x03_Odd_Even, J27 GS2, J28 GS2, J3 GS3, J4 GS2, J5 GS2, J6 GS3, J7 GS3, J8 GS2, J9 GS3, Q1 2N7002, U1 ADP1720ARMZ-5, U10 OPA2111KP, U11 AD8422ARMZ, U12 OP4117, U13 OPA2111KP, U14 AD8422ARMZ, U15 OP4117, U16 AD7173, U17 ADR445BR, U2 ADP1720ARMZ-3.3, U3 AD8475, U4 AD8475, U5 MAX7480ESA+, U6 MAX7480ESA+, U7 MAX7480ESA+, U8 MAX7480ESA+, U9 TLC555CD, Y1 FA-20H

Commit message: added decouple capacitors
Parts:
- moved R24 296.4 mm to (-87.8, 34.0)
- moved U13 296.1 mm to (-78.7, 26.4)
- moved J16 283.9 mm to (-14.5, -30.0), turned to 180 degrees
- moved U10 258.9 mm to (17.5, -40.2), turned to 90 degrees
- moved R34 240.4 mm to (58.3, -35.3)
- moved J8 236.5 mm to (39.1, -44.5)
- moved R35 230.4 mm to (59.4, -32.8)
- moved C42 214.6 mm to (57.0, -40.0), turned to 90 degrees
- moved R19 209.2 mm to (32.9, -47.8)
- moved R17 197.9 mm to (20.6, -36.6), turned to 90 degrees
- moved J7 196.2 mm to (22.6, -55.3), turned to 90 degrees
- moved J10 195.6 mm to (-67.6, 38.2)
- moved C29 189.7 mm to (25.9, -36.9)
- moved R30 187.8 mm to (39.1, -38.0), turned to 270 degrees
- moved R15 186.1 mm to (10.8, -40.6)
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Routing:
- net +12V: track 0.00 -> 107.8 mm
- net Net-(C40-Pad1): track 0.00 -> 52.0 mm
- net Net-(C20-Pad3): track 0.00 -> 35.8 mm
- net /Amplifier Block 1/IN+: track 0.00 -> 27.1 mm
- net GND: track 0.00 -> 26.9 mm
- net /Amplifier Block 1/IN-: track 0.00 -> 25.6 mm
- net Net-(C20-Pad1): track 0.00 -> 25.6 mm
- net Net-(J12-Pad3): track 0.00 -> 24.5 mm
- net Net-(C38-Pad1): track 0.00 -> 23.0 mm
- net Net-(C39-Pad1): track 0.00 -> 20.8 mm
- net -12V: track 0.00 -> 16.8 mm
- net Net-(C27-Pad2): track 0.00 -> 16.6 mm
- net Net-(J13-Pad3): track 0.00 -> 15.3 mm
- net Net-(C40-Pad2): track 0.00 -> 14.3 mm
- net Net-(C26-Pad2): track 0.00 -> 13.6 mm
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
Commit message: pcb layout for amplifier block
Parts:
- added J29: Teensy Port, Pin_Headers:Pin_Header_Straight_1x02_Pitch2.54mm, F.Cu at (-48.1, 109.4)
- added J30: GS3, Connectors:GS3, F.Cu at (-75.4, 84.0)
- added J31: GS3, Connectors:GS3, F.Cu at (-54.4, 84.0)
- added J32: Bluetooth, Pin_Headers:Pin_Header_Straight_1x06_Pitch2.54mm, F.Cu at (-87.2, 77.8)
- added J33: Reset Select, Connectors:GS3, F.Cu at (-37.2, 70.3)
- added J34: GS2, Connectors:GS2, F.Cu at (-24.7, 97.5)
- added J35: High Power, Pin_Headers:Pin_Header_Straight_1x02_Pitch2.54mm, F.Cu at (-73.9, 102.4)
- C10, C11, C12, C13, C20, C21: footprint Capacitors_SMD:C_0603_HandSoldering -> Neuro:Decouple_Cap_0603
- J17: value Conn_01x02 -> External
- J26: value Conn_02x03_Odd_Even -> ICSP Port
- R45, R48, R50: value R -> 2k
- R46, R47, R49: value R -> 1k
- moved C36 266.1 mm to (-10.1, -26.9), turned to 90 degrees
- moved J11 251.7 mm to (4.65, -19.9), turned to 90 degrees
- moved C46 237.1 mm to (10.8, -23.2), turned to 90 degrees
- moved R22 232.7 mm to (-14.5, -15.4)
- moved R37 220.0 mm to (33.5, -15.5), turned to 270 degrees
- moved R25 218.7 mm to (-5.05, -26.9), turned to 270 degrees
- moved R23 214.7 mm to (-14.5, -23.1)
- moved U14 213.9 mm to (10.7, -19.2)
- moved R28 213.0 mm to (16.4, -20.1)
- moved R40 208.0 mm to (30.6, -15.6), turned to 270 degrees
- moved C21 196.0 mm to (-13.4, -19.2), turned to 270 degrees
- moved R21 194.6 mm to (10.2, -36.3)
- moved C20 185.4 mm to (-13.2, -43.3), turned to 270 degrees
- moved J9 184.3 mm to (4.55, -26.9)
- moved R27 171.6 mm to (4.65, -18.1), turned to 180 degrees
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Connections:
- C10 pad 2: /RC Filter 1/GND -> GND
- C11 pad 2: /RC Filter 1/GND -> GND
- C22 pad 2: /ADConverter/GND -> GND
- C23 pad 2: /ADConverter/GND -> GND
- C24 pad 2: /ADConverter/GND -> GND
- C25 pad 2: /ADConverter/GND -> GND
- C31 pad 2: /ADConverter/GND -> GND
- C32 pad 2: /ADConverter/GND -> GND
- C48 pad 2: /ADConverter/GND -> GND
- C49 pad 2: /ADConverter/GND -> GND
- C50 pad 2: /ADConverter/GND -> GND
- C51 pad 2: /ADConverter/GND -> GND
- C52 pad 1: /ADConverter/VCC -> +5.5V
- C52 pad 2: /ADConverter/GND -> GND
- C63 pad 1: /USB Power/+5V -> +5V
- C63 pad 2: /USB Power/GND -> GND
- J1 pad 1: (no net) -> +5.5V
- J17 pad 2: /USB Power/GND -> GND
- J18 pad 5: /USB Power/GND -> GND
- J18 pad 6: /USB Power/GND -> GND
- J19 pad 2: /USB Power/+5V -> +5V
- J25 pad 1: (no net) -> CS
- J25 pad 2: (no net) -> /ADConverter/CS
- J26 pad 1: (no net) -> MOSI
- J26 pad 2: (no net) -> VCC
- J26 pad 3: (no net) -> SCL
- J26 pad 4: (no net) -> MISO
- J26 pad 5: (no net) -> /SPI Connector/RST
- J26 pad 6: (no net) -> GND
- J27 pad 1: (no net) -> SCL
- J27 pad 2: (no net) -> /ADConverter/SCL
- J28 pad 1: (no net) -> MISO
- J28 pad 2: (no net) -> /ADConverter/DI
- L2 pad 2: /ADConverter/VCC -> +5.5V
- R45 pad 1: (no net) -> /ADConverter/SCL
- R45 pad 2: (no net) -> GND
- R46 pad 1: (no net) -> SCL
- R46 pad 2: (no net) -> /ADConverter/SCL
- R47 pad 1: (no net) -> CS
- R47 pad 2: (no net) -> /ADConverter/CS
- R48 pad 1: (no net) -> /ADConverter/CS
- R48 pad 2: (no net) -> GND
- R49 pad 1: (no net) -> MISO
- R49 pad 2: (no net) -> /ADConverter/DI
- R50 pad 1: (no net) -> /ADConverter/DI
- R50 pad 2: (no net) -> GND
- U16 pad 14: (no net) -> MOSI
- U16 pad 15: (no net) -> /ADConverter/DI
- U16 pad 16: (no net) -> /ADConverter/SCL
- U16 pad 21: /ADConverter/GND -> GND
- U16 pad 39: /ADConverter/GND -> GND
- U16 pad 41: /ADConverter/GND -> GND
- U16 pad 8: /ADConverter/GND -> GND
- U17 pad 4: /ADConverter/GND -> GND
- Y1 pad 2: /ADConverter/GND -> GND
- Y1 pad 4: /ADConverter/GND -> GND
Routing:
- net -12V: track 16.8 -> 123.1 mm, vias 0 -> 5
- net Net-(C43-Pad1): track 0.00 -> 39.2 mm
- net Net-(J15-Pad3): track 0.00 -> 34.9 mm
- net Net-(C45-Pad1): track 0.00 -> 29.7 mm, vias 0 -> 2
- net Net-(C21-Pad1): track 0.00 -> 29.5 mm
- net Net-(C21-Pad3): track 0.00 -> 29.1 mm
- net Net-(J10-Pad2): track 0.00 -> 23.9 mm
- net Net-(C34-Pad1): track 0.00 -> 22.1 mm
- net Net-(J13-Pad1): track 0.00 -> 20.9 mm
- net Net-(C40-Pad1): track 52.0 -> 31.2 mm, vias 0 -> 2
- net Net-(J15-Pad1): track 0.00 -> 20.6 mm
- net Net-(C33-Pad1): track 0.00 -> 18.8 mm
- net /Amplifier Block 1/IN+: track 27.1 -> 9.28 mm
- net Net-(J13-Pad3): track 15.3 -> 32.5 mm
- net /Amplifier Block 2/IN+: track 0.00 -> 16.8 mm
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- added copper zone on B.Cu, net GND
Other:
- board outline added: 88.8 x 52.5 mm

Commit message: feat: power circuitry
Parts:
- added J36: 12 Volts, Pin_Headers:Pin_Header_Straight_1x02_Pitch2.54mm, F.Cu at (-20.6, -19.1)
- moved J19 233.9 mm to (-15.8, -53.3), turned to 180 degrees
- moved C55 216.9 mm to (34.5, -32.0)
- moved J17 207.2 mm to (-15.8, -49.8), turned to 90 degrees
- moved C57 203.3 mm to (34.5, -29.8)
- moved C56 200.0 mm to (37.9, -32.0)
- moved J18 193.3 mm to (-22.0, -51.4), turned to 270 degrees
- moved C1 192.0 mm to (39.4, -12.2), turned to 270 degrees
- moved C63 183.5 mm to (-13.2, -54.0), turned to 90 degrees
- moved C2 183.3 mm to (40.0, -7.80), turned to 180 degrees
- moved R1 172.0 mm to (40.0, -9.65), turned to 180 degrees
- moved C3 169.5 mm to (44.0, -7.80)
- moved U1 165.3 mm to (47.5, -10.0), turned to 270 degrees
- moved C4 164.8 mm to (55.0, -8.55), turned to 270 degrees
- moved J1 161.7 mm to (37.3, -13.0), turned to 180 degrees
- moved C5 153.7 mm to (47.8, -14.2)
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Routing:
- net GND: track 17.4 -> 93.2 mm, vias 20 -> 27
- net +12V: track 95.7 -> 168.8 mm, vias 5 -> 7
- net +5.5V: track 0.00 -> 66.7 mm
- net -12V: track 123.1 -> 163.6 mm, vias 5 -> 6
- net /External Power/VIN: track 0.00 -> 27.8 mm
- net +5V: track 0.00 -> 8.14 mm
- net Net-(C1-Pad1): track 0.00 -> 7.61 mm
- net Net-(J18-Pad1): track 0.00 -> 5.64 mm
- net +3V: track 0.00 -> 4.67 mm
- net Net-(J17-Pad1): track 0.00 -> 2.28 mm
- net Net-(D1-Pad1): track 0.00 -> 1.75 mm
- net Net-(C20-Pad1): track 28.6 -> 27.8 mm
- net Net-(C21-Pad3): track 29.1 -> 28.6 mm

Commit message: feat: attenuator and clock circuits
Parts:
- moved J32 358.5 mm to (270.4, 102.5)
- moved J30 343.2 mm to (265.4, 43.1)
- moved J31 315.6 mm to (257.8, 130.5)
- moved J34 295.8 mm to (269.4, 66.5)
- moved J29 289.7 mm to (238.9, 148.8)
- moved C9 233.1 mm to (42.2, -30.0), turned to 270 degrees
- moved U3 215.8 mm to (42.2, -39.6), turned to 90 degrees
- moved U4 214.6 mm to (42.2, -21.9), turned to 90 degrees
- moved C12 206.5 mm to (184.1, -7.62)
- moved R10 189.1 mm to (147.8, -35.9)
- moved J33 186.8 mm to (149.1, 84.8)
- moved C7 184.6 mm to (37.1, -39.6), turned to 90 degrees
- moved C10 183.8 mm to (128.8, -39.5)
- moved C17 166.0 mm to (143.9, -9.10)
- moved C19 162.9 mm to (57.3, -14.8), turned to 90 degrees
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Routing:
- net +5V: track 8.14 -> 183.2 mm, vias 0 -> 3
- net VCCIO: track 0.00 -> 41.9 mm, vias 0 -> 3
- net /Attenuator/+IN0.4XB: track 0.00 -> 39.7 mm
- net /Attenuator/+IN0.4XA: track 0.00 -> 36.4 mm
- net /Attenuator/-IN0.4XA: track 0.00 -> 34.5 mm, vias 0 -> 2
- net /Attenuator/-IN0.4XB: track 0.00 -> 30.8 mm, vias 0 -> 2
- net Net-(C9-Pad1): track 0.00 -> 22.7 mm, vias 0 -> 2
- net GND: track 93.2 -> 109.8 mm, vias 27 -> 33
- net Net-(C19-Pad1): track 0.00 -> 11.9 mm, vias 0 -> 2
- net Net-(J3-Pad1): track 0.00 -> 11.6 mm
- net Net-(R6-Pad2): track 0.00 -> 9.50 mm
- net Net-(J3-Pad3): track 0.00 -> 7.81 mm
- net Net-(C18-Pad1): track 0.00 -> 3.50 mm
Other:
- board size 88.8 x 52.5 mm -> 108.6 x 52.5 mm

Commit message: feat: filter circuits
refactor
Parts:
- U5, U6, U7, U8: footprint Housings_SOIC:SO-8_5.3x6.2mm_Pitch1.27mm -> Housings_SOIC:SOIC-8_3.9x4.9mm_Pitch1.27mm
- moved R48 233.5 mm to (242.8, 108.4)
- moved R47 207.8 mm to (238.3, 108.4)
- moved R45 205.2 mm to (245.4, 103.9), turned to 180 degrees
- moved J25 190.6 mm to (238.3, 110.8), turned to 90 degrees
- moved R46 183.8 mm to (249.8, 103.9), turned to 180 degrees
- moved R49 157.1 mm to (261.4, 103.9)
- moved J27 150.5 mm to (249.8, 101.5), turned to 270 degrees
- moved R12 145.4 mm to (122.4, 100.4), turned to 270 degrees
- moved C1 143.2 mm to (104.9, 115.0)
- moved C18 143.2 mm to (129.3, 118.7)
- moved C19 143.2 mm to (122.8, 112.4)
- moved C2 143.2 mm to (105.5, 119.5)
- moved C20 143.2 mm to (52.4, 84.0)
- moved C21 143.2 mm to (52.1, 108.1)
- moved C26 143.2 mm to (63.1, 76.8)
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Routing:
- net /Clock Block/CLK: track 0.00 -> 98.2 mm
- net +5V: track 183.2 -> 267.0 mm, vias 3 -> 13
- net /Attenuator/+OUTA: track 0.00 -> 34.5 mm, vias 0 -> 2
- net GND: track 109.8 -> 139.5 mm, vias 33 -> 40
- net /Attenuator/+OUTB: track 0.00 -> 28.9 mm, vias 0 -> 2
- net /Attenuator/-OUTA: track 0.00 -> 18.5 mm
- net /ADConverter/AIN4: track 0.00 -> 18.3 mm, vias 0 -> 2
- net /ADConverter/AIN6: track 0.00 -> 15.9 mm, vias 0 -> 2
- net /Attenuator/-OUTB: track 0.00 -> 15.7 mm
- net Net-(C15-Pad1): track 0.00 -> 14.0 mm, vias 0 -> 2
- net Net-(C16-Pad1): track 0.00 -> 13.9 mm, vias 0 -> 2
- net Net-(C17-Pad1): track 0.00 -> 13.8 mm, vias 0 -> 2
- net Net-(C14-Pad1): track 0.00 -> 13.4 mm, vias 0 -> 2
- net /ADConverter/AIN5: track 0.00 -> 13.0 mm
- net /ADConverter/AIN7: track 0.00 -> 11.5 mm
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Other:
- board size 108.6 x 52.5 mm -> 124.9 x 52.6 mm

Commit message: feat: ADC Circuit
Parts:
- added U18: Arduino, Pin_Headers:Pin_Header_Straight_2x12_Pitch2.54mm, F.Cu at (185.1, 123.0)
- moved J28 71.7 mm to (197.9, 73.7), turned to 270 degrees
- moved J32 71.3 mm to (198.8, 110.3), turned to 90 degrees
- moved R49 66.5 mm to (202.2, 73.7)
- moved R50 65.9 mm to (206.8, 75.1), turned to 270 degrees
- moved C24 62.8 mm to (208.8, 86.4)
- moved U17 62.2 mm to (208.8, 98.5), turned to 90 degrees
- moved J30 62.0 mm to (206.3, 106.8), turned to 90 degrees
- moved C22 61.8 mm to (208.1, 91.5), turned to 90 degrees
- moved C23 61.5 mm to (205.8, 91.4), turned to 90 degrees
- moved J25 61.4 mm to (188.7, 74.6), turned to 270 degrees
- moved C50 60.8 mm to (211.2, 103.0), turned to 0 degrees
- moved J26 60.2 mm to (198.5, 79.1), turned to 90 degrees
- moved C51 59.0 mm to (211.2, 104.8), turned to 0 degrees
- moved R48 58.5 mm to (193.3, 77.2)
- moved C52 58.3 mm to (211.3, 107.0), turned to 0 degrees
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Connections:
- J20 pad 1: (no net) -> AD3
- J21 pad 1: (no net) -> AD2
- J22 pad 1: (no net) -> AD1
- J23 pad 1: (no net) -> AD0
- J30 pad 1: (no net) -> RxI
- J33 pad 1: (no net) -> Net-(J33-Pad1)
- J33 pad 3: (no net) -> Net-(J33-Pad3)
- J34 pad 2: (no net) -> Net-(J34-Pad2)
- Q1 pad 1: (no net) -> EXCLK
- R44 pad 2: (no net) -> Net-(R44-Pad2)
Routing:
- net Net-(R6-Pad2): track 9.50 -> 16.7 mm
- net Net-(C19-Pad1): track 11.9 -> 13.1 mm
Other:
- board size 124.9 x 52.6 mm -> 124.9 x 52.5 mm

Commit message: refactor: route improvements
Parts:
- moved J27 0.53 mm to (199.2, 84.0)
Connections:
- J31 pad 1: TxO -> RxI
Routing:
- net CS: track 0.00 -> 118.3 mm, vias 0 -> 3
- net +5.5V: track 66.7 -> 181.8 mm, vias 0 -> 4
- net MISO: track 0.00 -> 108.9 mm, vias 0 -> 2
- net SCL: track 0.00 -> 104.0 mm, vias 0 -> 2
- net MOSI: track 0.00 -> 103.3 mm, vias 0 -> 3
- net GND: track 139.5 -> 235.5 mm, vias 40 -> 47
- net AD3: track 0.00 -> 90.2 mm, vias 0 -> 2
- net AD1: track 0.00 -> 86.1 mm, vias 0 -> 2
- net Net-(J33-Pad1): track 0.00 -> 80.7 mm, vias 0 -> 1
- net +3V: track 4.67 -> 78.3 mm, vias 0 -> 2
- net VCCIO: track 41.9 -> 114.7 mm, vias 3 -> 5
- net VCC: track 0.00 -> 64.9 mm, vias 0 -> 4
- net AD0: track 0.00 -> 59.6 mm, vias 0 -> 2
- net TxO: track 0.00 -> 53.3 mm, vias 0 -> 3
- net AD2: track 0.00 -> 50.6 mm
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Other:
- board size 124.9 x 52.5 mm -> 127 x 53.6 mm
- net class Default: clearance 0.2 -> 0.1
- rule trace_clearance: 0.2 -> 0.1
- rule trace_min: 0.2 -> 0.1
- rule via_min_size: 0.4 -> 0.3

Commit message: optimize: routing and placement
optimize: squeeze space

optimize: squeeze space contd.

optimize: contd.
Parts:
- removed J11: GS2, Connectors:GS2
- removed J29: Teensy Port, Pin_Headers:Pin_Header_Straight_1x02_Pitch2.54mm
- removed J35: High Power, Pin_Headers:Pin_Header_Straight_1x02_Pitch2.54mm
- removed J36: 12 Volts, Pin_Headers:Pin_Header_Straight_1x02_Pitch2.54mm
- added REF***: ESD-Logo_6.6x6mm_SilkScreen, Symbols:ESD-Logo_6.6x6mm_SilkScreen, F.Cu at (140.8, 81.5)
- J8: value GS2 -> PowerOut; footprint Connectors:GS2 -> Pin_Headers:Pin_Header_Straight_2x02_Pitch2.54mm
- moved C53 55.4 mm to (99.3, 114.4), turned to 270 degrees
- moved C55 52.4 mm to (101.7, 114.4), turned to 270 degrees
- moved C57 49.4 mm to (104.0, 114.4), turned to 270 degrees
- moved C59 46.5 mm to (106.3, 114.4), turned to 270 degrees
- moved C61 43.6 mm to (108.7, 114.4), turned to 270 degrees
- moved C54 40.5 mm to (116.2, 79.9), turned to 270 degrees
- moved C56 39.3 mm to (118.5, 79.9), turned to 270 degrees
- moved C58 38.3 mm to (120.7, 79.9), turned to 270 degrees
- moved C60 37.6 mm to (123.0, 79.9), turned to 270 degrees
- moved C62 37.2 mm to (125.2, 79.9), turned to 270 degrees
- moved J8 36.1 mm to (93.2, 107.7), turned to 0 degrees
- moved R11 32.4 mm to (155.1, 85.7), turned to 90 degrees
- moved R13 32.3 mm to (155.1, 102.0), turned to 90 degrees
- moved U7 31.7 mm to (149.6, 85.2)
- moved U8 31.5 mm to (149.6, 101.4)
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Connections:
- J16 pad 1: GND -> /Amplifier Block 2/IN+
- J16 pad 2: /Amplifier Block 2/IN+ -> /Amplifier Block 2/IN-
- J16 pad 3: /Amplifier Block 2/IN- -> GND
- J16 pad 4: /Amplifier Block 1/IN- -> GND
- J16 pad 6: GND -> /Amplifier Block 1/IN-
- J8 pad 1: Net-(J8-Pad1) -> -12V
- J8 pad 2: Net-(J8-Pad2) -> +12V
- R19 pad 2: Net-(J8-Pad1) -> Net-(R19-Pad2)
- R27 pad 2: Net-(J11-Pad1) -> Net-(R27-Pad2)
- U11 pad 2: Net-(J8-Pad2) -> Net-(R19-Pad2)
- U14 pad 2: Net-(J11-Pad2) -> Net-(R27-Pad2)
Routing:
- net (no net): track 0.00 -> 140.0 mm, vias 0 -> 14
- net +5V: track 294.6 -> 352.0 mm, vias 15 -> 23
- net /Clock Block/CLK: track 98.2 -> 134.0 mm, vias 0 -> 4
- net /Attenuator/+OUTA: track 34.5 -> 14.7 mm, vias 2 -> 0
- net /Attenuator/+IN0.4XA: track 36.4 -> 17.7 mm
- net /Attenuator/-IN0.4XA: track 34.5 -> 15.8 mm, vias 2 -> 0
- net /Attenuator/+IN0.4XB: track 39.7 -> 21.3 mm
- net Net-(J13-Pad3): track 32.5 -> 15.1 mm
- net Net-(J15-Pad3): track 34.9 -> 18.4 mm
- net Net-(C43-Pad1): track 39.2 -> 22.8 mm
- net /Attenuator/-IN0.4XB: track 30.8 -> 15.9 mm, vias 2 -> 0
- net /Attenuator/+OUTB: track 28.9 -> 14.5 mm, vias 2 -> 0
- net Net-(C38-Pad1): track 36.9 -> 22.5 mm
- net Net-(C40-Pad1): track 31.2 -> 16.9 mm, vias 2 -> 0
- net Net-(C44-Pad1): track 15.2 -> 29.4 mm
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Other:
- net class Default: clearance 0.1 -> 0.16
- rule trace_clearance: 0.1 -> 0.16
- rule trace_min: 0.1 -> 0.16
